File: kicad-files/extrimism.kicad_sch (KiCad schematic)
At the start: 31 parts, among them SW1 SW_Push, SW10 SW_Push, SW11 SW_Push, SW12 SW_Push, SW2 SW_Push, SW3 SW_Push, SW4 SW_Push, SW5 SW_Push, SW6 SW_Push, SW7 SW_Push, SW8 SW_Push, SW9 SW_Push, U1 Pico, U2 RFM95W-868S2

Commit message: updated PCB design
Parts:
- removed R12: 15k, Resistor_THT:R_Axial_DIN0309_L9.0mm_D3.2mm_P2.54mm_Vertical, symbol Device:R
- removed R8: 2.2k, Resistor_THT:R_Axial_DIN0309_L9.0mm_D3.2mm_P2.54mm_Vertical, symbol Device:R
- removed R9: 4k, Resistor_THT:R_Axial_DIN0309_L9.0mm_D3.2mm_P2.54mm_Vertical, symbol Device:R
- added C1, C2: 10nF, Capacitor_THT:C_Disc_D5.0mm_W2.5mm_P5.00mm, symbol Device:C
- added C3: 100uF, Capacitor_THT:C_Disc_D5.0mm_W2.5mm_P5.00mm, symbol Device:C
- added C4: 100nF, Capacitor_THT:C_Disc_D5.0mm_W2.5mm_P5.00mm, symbol Device:C
- added D1: 1N4001, Diode_THT:D_DO-41_SOD81_P10.16mm_Horizontal, symbol Diode:1N4001
- added D2: IR_LED, LED_THT:LED_D3.0mm, symbol Device:LED
- added H1, H2, H3: MountingHole, MountingHole:MountingHole_2.1mm, symbol Mechanical:MountingHole
- added Q1: NPN, Package_TO_SOT_THT:TO-92_Inline, symbol Simulation_SPICE:NPN
- added U1: TSOP38238, OptoDevice:Vishay_MINICAST-3Pin, symbol Interface_Optical:TSOP382xx
- BC1: footprint rfm95:Adafruit_259 -> extrimism_lib:extrimism_lib
- R1, R7: footprint Resistor_THT:R_Axial_DIN0309_L9.0mm_D3.2mm_P2.54mm_Vertical -> Resistor_THT:R_Axial_DIN0207_L6.3mm_D2.5mm_P7.62mm_Horizontal
- R10: value 6.8k -> 470; footprint Resistor_THT:R_Axial_DIN0309_L9.0mm_D3.2mm_P2.54mm_Vertical -> Resistor_THT:R_Axial_DIN0207_L6.3mm_D2.5mm_P7.62mm_Horizontal
- R11: value 10k -> 0; footprint Resistor_THT:R_Axial_DIN0309_L9.0mm_D3.2mm_P2.54mm_Vertical -> Resistor_THT:R_Axial_DIN0207_L6.3mm_D2.5mm_P7.62mm_Horizontal
- R2: value 2.2k -> 1.2k; footprint Resistor_THT:R_Axial_DIN0309_L9.0mm_D3.2mm_P2.54mm_Vertical -> Resistor_THT:R_Axial_DIN0207_L6.3mm_D2.5mm_P7.62mm_Horizontal
- R3: value 4k -> 1.8k; footprint Resistor_THT:R_Axial_DIN0309_L9.0mm_D3.2mm_P2.54mm_Vertical -> Resistor_THT:R_Axial_DIN0207_L6.3mm_D2.5mm_P7.62mm_Horizontal
- R4: value 6.8k -> 2.7k; footprint Resistor_THT:R_Axial_DIN0309_L9.0mm_D3.2mm_P2.54mm_Vertical -> Resistor_THT:R_Axial_DIN0207_L6.3mm_D2.5mm_P7.62mm_Horizontal
- R5: value 10k -> 3.3k; footprint Resistor_THT:R_Axial_DIN0309_L9.0mm_D3.2mm_P2.54mm_Vertical -> Resistor_THT:R_Axial_DIN0207_L6.3mm_D2.5mm_P7.62mm_Horizontal
- R6: value 15k -> 4.7k; footprint Resistor_THT:R_Axial_DIN0309_L9.0mm_D3.2mm_P2.54mm_Vertical -> Resistor_THT:R_Axial_DIN0207_L6.3mm_D2.5mm_P7.62mm_Horizontal
- R8: renamed from R13; footprint Resistor_THT:R_Axial_DIN0309_L9.0mm_D3.2mm_P2.54mm_Vertical -> Resistor_THT:R_Axial_DIN0207_L6.3mm_D2.5mm_P7.62mm_Horizontal
- R9: renamed from R14; footprint Resistor_THT:R_Axial_DIN0309_L9.0mm_D3.2mm_P2.54mm_Vertical -> Resistor_THT:R_Axial_DIN0207_L6.3mm_D2.5mm_P7.62mm_Horizontal
- renumbered U1 to U2, U2 to U3
Connections:
- net GND: now also BC1.5 (load-), U2.18 (GND), U2.23 (GND), U2.28 (GND), U2.38 (GND), U3.1 (GND), C1.2, C2.2, C3.2, C4.2, D2.1 (K), Q1.3 (E), U1.2 (GND); no longer BZ1.2 (-)
- net adc0: now also SW1.1, SW2.1, SW3.1, SW4.1, SW5.1, SW6.1, C1.1; no longer R1.1, R2.1, R3.1, R4.1, R5.1, R6.1
- net adc1: now also SW10.2, SW11.2, SW12.2, SW7.2, SW8.2, SW9.2, C2.1; no longer R10.1, R11.1, R7.1
- net buzz: now also R7.1; no longer BZ1.1 (+)
- net at R3.2, SW3.2: now also R4.1, SW9.1
- net at R7.2: now also Q1.2 (B); no longer SW7.2
- net at R1.2, SW1.2: now also R2.1, SW7.1
- net at R11.2: now also U3.6 (RESET); no longer SW11.2
- net at U2.26 (GPIO20): now also R11.1; no longer U3.6 (RESET)
- net at R6.2, SW6.2: now also SW12.1
- net at R2.2, SW2.2: now also R3.1, SW8.1
- net at R10.2: now also D2.2 (A); no longer SW10.2
- net at R5.2, SW5.2: now also R6.1, SW11.1
- net at R4.2, SW4.2: now also R5.1, SW10.1
- net ir_tx: now reaches U2.19 (GPIO14)
- net ir_tx: now also R10.1
- net ir_rx: now reaches U2.20 (GPIO15)
- net ir_rx: now also U1.1 (OUT)
- removed net 3v3_kb: SW1.1, SW10.1, SW11.1, SW12.1, SW2.1, SW3.1, SW4.1, SW5.1, SW6.1, SW7.1, SW8.1, SW9.1, U2.36 (3V3), U3.13 (3.3V)
- new net: BZ1.2 (-), D1.2 (A), Q1.1 (C)
- new net 3v3: BZ1.1 (+), C3.1, C4.1, D1.1 (K), R1.1, U1.3 (Vs), U2.36 (3V3), U3.13 (3.3V)
- no-connect marks 41 -> 35
Other:
- note added: "IR Stuff"
- note added: "Mounts"
- moved on the sheet: BC1, BZ1, SW1, SW10, SW11, SW12, SW3, SW4, SW5, SW6, SW7, SW8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
